File: heart-files/keyboard.kicad_sch (KiCad schematic)
At the start: 168 parts

Commit message: update but atp I'm going to start from scratch the correct way lowkey
Parts:
- added A1: RaspberryPi_Pico, Module:RaspberryPi_Pico_Common_Unspecified, symbol MCU_Module:RaspberryPi_Pico
- added JS1: joystick_analog, PCM_marbastlib-various:joystick_psp1000, symbol PCM_marbastlib-various:joystick_analog
Connections:
- net col0: now also A1.1 (GPIO0)
- new net: A1.13 (GND), A1.18 (GND), A1.23 (GND), A1.28 (GND), A1.3 (GND), A1.38 (GND), A1.8 (GND), JS1.2 (GND)
- new net: A1.32 (GPIO27_ADC1), JS1.1 (X)
- new net: A1.34 (GPIO28_ADC2), JS1.3 (Y)
- new net: A1.36 (3V3), JS1.4 (VCC)
